Commit message: Umut

File: src/wheelchair/urdf/wheelchair.urdf (robot description, URDF)
Before this commit: robot wheelchair, 22 links, 21 joints
Links:
- removed link back_pole
- removed link back_seat
- removed link base_footprint
- removed link block2_seat
- removed link block3_seat
- removed link front_caster_left
- removed link front_caster_right
- removed link front_pole_left
- removed link front_pole_right
- removed link front_wheel_left
- removed link front_wheel_right
- removed link laser
- removed link left_rear_wheel
- removed link lidar_panel
- removed link right_rear_wheel
- removed link rs_lidar_link
- removed link side_seat
- removed link side_seat_2
- removed link soft_seat
- added link camera, mass 0.0247927918584364; collision mesh filename=package://wheelchair_urdf/meshes/camera.STL; visual mesh filename=package://wheelchair_urdf/meshes/camera.STL
- added link left_big_wheel, mass 3.19005851775017; collision mesh filename=package://wheelchair_urdf/meshes/left_big_wheel.STL; visual mesh filename=package://wheelchair_urdf/meshes/left_big_wheel.STL
- added link left_small_wheel, mass 1.31881639542862; collision mesh filename=package://wheelchair_urdf/meshes/left_small_wheel.STL; visual mesh filename=package://wheelchair_urdf/meshes/left_small_wheel.STL
- added link right_big_wheel, mass 3.19005851775017; collision mesh filename=package://wheelchair_urdf/meshes/right_big_wheel.STL; visual mesh filename=package://wheelchair_urdf/meshes/right_big_wheel.STL
- added link right_smaal_wheel, mass 1.31881639542862; collision mesh filename=package://wheelchair_urdf/meshes/right_smaal_wheel.STL; visual mesh filename=package://wheelchair_urdf/meshes/right_smaal_wheel.STL
- link base_link: mass 1.0 -> 100.569950446923; geometry collision mesh filename=package://wheelchair_urdf/meshes/base_link.STL; visual mesh filename=package://wheelchair_urdf/meshes/base_link.STL
- link rp_laser_back: mass 1.0 -> 0.165382757413928; geometry collision mesh filename=package://wheelchair_urdf/meshes/rp_laser_back.STL; visual mesh filename=package://wheelchair_urdf/meshes/rp_laser_back.STL
- link rp_laser_front: mass 0.1 -> 0.165382782759051; geometry collision mesh filename=package://wheelchair_urdf/meshes/rp_laser_front.STL; visual mesh filename=package://wheelchair_urdf/meshes/rp_laser_front.STL
Joints:
- removed joint back_pole_joint
- removed joint back_seat_joint
- removed joint base_joint
- removed joint block2_joint
- removed joint block3_joint
- removed joint camera_link_joint
- removed joint front_caster_left_joint
- removed joint front_caster_right_joint
- removed joint front_pole_left_joint
- removed joint front_pole_right_joint
- removed joint front_wheel_left_joint
- removed joint front_wheel_right_joint
- removed joint laser_joint
- removed joint left_rear_wheel_joint
- removed joint lidar_panel_joint
- removed joint right_rear_wheel_joint
- removed joint side_seat_2_joint
- removed joint side_seat_joint
- removed joint soft_joint
- added joint camera_joint: type fixed, parent base_link, child camera, origin xyz=-0.387035971879652 -0.00396906785592691 1.52648295547757 rpy=0 0 0, axis -0.99739 -0.072202 0, limit lower=0 upper=0 effort=0 velocity=0
- added joint left_big_wheel_joint: type continuous, parent base_link, child left_big_wheel, origin xyz=-0.32005 0.315 -0.008 rpy=0 0 0, axis 0 -1 0, limit effort=1 velocity=1
- added joint left_small_wheel_joint: type revolute, parent base_link, child left_small_wheel, origin xyz=0.31993 0.2835 -0.073 rpy=0 0 0.00055161, axis 0 1 0, limit lower=0 upper=0 effort=0 velocity=0
- added joint right_big_wheel_joint: type continuous, parent base_link, child right_big_wheel, origin xyz=-0.32005 -0.315 -0.008 rpy=0 0 0, axis 0 -1 0, limit effort=1 velocity=1
- added joint right_small_wheel_joint: type revolute, parent base_link, child right_smaal_wheel, origin xyz=0.31978 -0.2835 -0.073 rpy=0 0 0, axis 0.0043627 0.99999 0, limit lower=0 upper=0 effort=0 velocity=0
- joint rp_laser_back_joint: origin xyz=0.245 0.086 0.325 rpy=0 0 0 -> xyz=-0.36833 0.305 0.25299 rpy=0 0 -0.436332
- joint rp_laser_front_joint: origin xyz=0 -0.125 -0.245 rpy=0 0 -1.57 -> xyz=0.4012 -3.7661E-05 -0.092559 rpy=0 0 0.00055161; parent lidar_panel -> base_link
