Commit message: Umut

File: src/wheel_chair/urdf/wheel_chair.urdf (robot description, URDF)
Before this commit: robot wheel_chair, 8 links, 7 joints
Links:
- removed link back_lidar
- removed link front_lidar
- added link rp_laser_back, mass 0.165382757413928; collision mesh filename=package://wheel_chair/meshes/rp_laser_back.STL; visual mesh filename=package://wheel_chair/meshes/rp_laser_back.STL
- added link rp_laser_front, mass 0.165382782759051; collision mesh filename=package://wheel_chair/meshes/rp_laser_front.STL; visual mesh filename=package://wheel_chair/meshes/rp_laser_front.STL
Joints:
- removed joint back_lidar_joint
- removed joint front_lidar_joint
- added joint rp_laser_back_joint: type fixed, parent base_link, child rp_laser_back, origin xyz=-0.36833 0.305 0.25299 rpy=0 0 0, axis 0 0 0
- added joint rp_laser_front_joint: type fixed, parent base_link, child rp_laser_front, origin xyz=0.4012 -3.7661E-05 -0.092559 rpy=0 0 0.00055161, axis 0 0 0

Commit message: Umut

File: src/wheel_chair/urdf/wheel_chair.urdf (robot description, URDF)
Before this commit: robot wheel_chair, 8 links, 7 joints
Joints:
- joint rp_laser_back_joint: origin xyz=-0.36833 0.305 0.25299 rpy=0 0 0 -> xyz=-0.36833 0.305 0.25299 rpy=0 0 -0.4
